File: Keyboard_PCB/usb.kicad_sch (KiCad schematic)
At the start: 0 parts

Commit message: Schematic V1
Parts:
- added FL1: TDK ACM2012-900, ACM2012_900_2P_T002:ACM2012_TDK, symbol Filter:Choke_Coilcraft_0603USB-222
- added J1: USB-C 16P, Connector_USB:USB_C_Receptacle_HCTL_HC-TYPE-C-16P-01A, symbol Connector:USB_C_Receptacle_USB2.0_16P
- added R1: 5k1, Resistor_SMD:R_0603_1608Metric, symbol Device:R_Small
- added U2: USBLC6-2SC6, Package_TO_SOT_SMD:SOT-23-6, symbol Power_Protection:USBLC6-2SC6
Connections:
- new net: FL1.1, U2.6 (I/O1)
- new net: FL1.4, U2.4 (I/O2)
- new net: J1.A5 (CC1), J1.B5 (CC2), R1.2
- new net: J1.A7 (D-), J1.B7 (D-), U2.1 (I/O1)
- new net: J1.A6 (D+), J1.B6 (D+), U2.3 (I/O2)
- new net +5V: J1.A4 (VBUS), J1.A9 (VBUS), J1.B4 (VBUS), J1.B9 (VBUS), U2.5 (VBUS)
- new net GND: J1.A1 (GND), J1.A12 (GND), J1.B1 (GND), J1.B12 (GND), R1.1, U2.2 (GND)
- new net USB_DN: FL1.2
- new net USB_DP: FL1.3
- no-connect marks 0 -> 3
Other:
- note added: "CC1"
- note added: "CC2"
