File: Keyboard_PCB/usb.kicad_sch (KiCad schematic)
At the start: 4 parts, among them J1 USB-C 16P, U2 USBLC6-2SC6

Commit message: OLD version final commit
Parts:
- FL1: value TDK ACM2012-900 -> TDK ACM2012-900
Changed lines of the file:
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@@
 			)
 		)
-		(property "Value" " TDK ACM2012-900"
+		(property "Value" "TDK ACM2012-900"
 			(at 80.01 43.942 0)
 			(effects
