File: Keyboard_PCB/grid.kicad_sch (KiCad schematic)
At the start: 0 parts

Commit message: Schematic V1
Parts:
- added D1, D10, D11, D12, D13, D14, D15, D16, D17, D18, D19, D2, D20, D21, D22, D23, D24, D25, D26, D27, D28, D29, D3, D30, D31, D32, D33, D34, D35, D36, D37, D38, D39, D4, D40, D41, D42, D43, D44, D45, D46, D47, D48, D49, D5, D50, D51, D52, D53, D54, D55, D56, D57, D58, D59, D6, D60, D61, D62, D63, D64, D65, D66, D67, D68, D7, D8, D9: D_Small, symbol Device:D_Small
- added SW1: ESC, symbol Switch:SW_Push_45deg
- added SW10: 9, symbol Switch:SW_Push_45deg
- added SW11: 0, symbol Switch:SW_Push_45deg
- added SW12: -, symbol Switch:SW_Push_45deg
- added SW13: =, symbol Switch:SW_Push_45deg
- added SW14: <-, symbol Switch:SW_Push_45deg
- added SW15: DEL, symbol Switch:SW_Push_45deg
- added SW16: TAB, symbol Switch:SW_Push_45deg
- added SW17: Q, symbol Switch:SW_Push_45deg
- added SW18: W, symbol Switch:SW_Push_45deg
- added SW19: E, symbol Switch:SW_Push_45deg
- added SW2: 1, symbol Switch:SW_Push_45deg
- added SW20: R, symbol Switch:SW_Push_45deg
- added SW21: T, symbol Switch:SW_Push_45deg
- added SW22: Y, symbol Switch:SW_Push_45deg
- added SW23: U, symbol Switch:SW_Push_45deg
- added SW24: I, symbol Switch:SW_Push_45deg
- added SW25: O, symbol Switch:SW_Push_45deg
- added SW26: P, symbol Switch:SW_Push_45deg
- added SW27: [, symbol Switch:SW_Push_45deg
- added SW28: ], symbol Switch:SW_Push_45deg
- added SW29: \, symbol Switch:SW_Push_45deg
- added SW3: 2, symbol Switch:SW_Push_45deg
- added SW30: HOME, symbol Switch:SW_Push_45deg
- added SW31: CAPS, symbol Switch:SW_Push_45deg
- added SW32: A, symbol Switch:SW_Push_45deg
- added SW33: S, symbol Switch:SW_Push_45deg
- added SW34: D, symbol Switch:SW_Push_45deg
- added SW35: F, symbol Switch:SW_Push_45deg
- added SW36: G, symbol Switch:SW_Push_45deg
- added SW37: H, symbol Switch:SW_Push_45deg
- added SW38: J, symbol Switch:SW_Push_45deg
- added SW39: K, symbol Switch:SW_Push_45deg
- added SW4: 3, symbol Switch:SW_Push_45deg
- added SW40: L, symbol Switch:SW_Push_45deg
- added SW41: ;, symbol Switch:SW_Push_45deg
- added SW42: ', symbol Switch:SW_Push_45deg
- added SW43: ENTER, symbol Switch:SW_Push_45deg
- added SW44: PG_U, symbol Switch:SW_Push_45deg
- added SW45, SW56: SHIFT, symbol Switch:SW_Push_45deg
- added SW46: Z, symbol Switch:SW_Push_45deg
- added SW47: X, symbol Switch:SW_Push_45deg
- added SW48: C, symbol Switch:SW_Push_45deg
- added SW49: V, symbol Switch:SW_Push_45deg
- added SW5: 4, symbol Switch:SW_Push_45deg
- added SW50: B, symbol Switch:SW_Push_45deg
- added SW51: N, symbol Switch:SW_Push_45deg
- added SW52: M, symbol Switch:SW_Push_45deg
- added SW53: ,, symbol Switch:SW_Push_45deg
- added SW54: ., symbol Switch:SW_Push_45deg
- added SW55: /, symbol Switch:SW_Push_45deg
- added SW57: UP, symbol Switch:SW_Push_45deg
- added SW58: PG_D, symbol Switch:SW_Push_45deg
- added SW59, SW65: CTRL, symbol Switch:SW_Push_45deg
- added SW6: 5, symbol Switch:SW_Push_45deg
- added SW60, SW64: CODE, symbol Switch:SW_Push_45deg
- added SW61, SW63: ALT, symbol Switch:SW_Push_45deg
- added SW62: SPACE, symbol Switch:SW_Push_45deg
- added SW66: LEFT, symbol Switch:SW_Push_45deg
- added SW67: DOWN, symbol Switch:SW_Push_45deg
- added SW68: RIGHT, symbol Switch:SW_Push_45deg
- added SW7: 6, symbol Switch:SW_Push_45deg
- added SW8: 7, symbol Switch:SW_Push_45deg
- added SW9: 8, symbol Switch:SW_Push_45deg
Connections:
- net COL_0: now also SW1.1, SW16.1, SW31.1, SW45.1, SW59.1
- net COL_1: now also SW17.1, SW2.1, SW32.1, SW46.1, SW60.1
- net COL_10: now also SW11.1, SW26.1, SW41.1, SW55.1, SW65.1
- net COL_11: now also SW12.1, SW27.1, SW42.1, SW56.1, SW66.1
- net COL_12: now also SW13.1, SW28.1
- net COL_13: now also SW14.1, SW29.1, SW43.1, SW57.1, SW67.1
- net COL_14: now also SW15.1, SW30.1, SW44.1, SW58.1, SW68.1
- net COL_2: now also SW18.1, SW3.1, SW33.1, SW47.1, SW61.1
- net COL_3: now also SW19.1, SW34.1, SW4.1, SW48.1
- net COL_4: now also SW20.1, SW35.1, SW49.1, SW5.1
- net COL_5: now also SW21.1, SW36.1, SW50.1, SW6.1, SW62.1
- net COL_6: now also SW22.1, SW37.1, SW51.1, SW7.1
- net COL_7: now also SW23.1, SW38.1, SW52.1, SW8.1
- net COL_8: now also SW24.1, SW39.1, SW53.1, SW63.1, SW9.1
- net COL_9: now also SW10.1, SW25.1, SW40.1, SW54.1, SW64.1
- net ROW_0: now also D1.1 (K), D10.1 (K), D11.1 (K), D12.1 (K), D13.1 (K), D14.1 (K), D15.1 (K), D2.1 (K), D3.1 (K), D4.1 (K), D5.1 (K), D6.1 (K), D7.1 (K), D8.1 (K), D9.1 (K)
- net ROW_1: now also D16.1 (K), D17.1 (K), D18.1 (K), D19.1 (K), D20.1 (K), D21.1 (K), D22.1 (K), D23.1 (K), D24.1 (K), D25.1 (K), D26.1 (K), D27.1 (K), D28.1 (K), D29.1 (K), D30.1 (K)
- net ROW_2: now also D31.1 (K), D32.1 (K), D33.1 (K), D34.1 (K), D35.1 (K), D36.1 (K), D37.1 (K), D38.1 (K), D39.1 (K), D40.1 (K), D41.1 (K), D42.1 (K), D43.1 (K), D44.1 (K)
- net ROW_3: now also D45.1 (K), D46.1 (K), D47.1 (K), D48.1 (K), D49.1 (K), D50.1 (K), D51.1 (K), D52.1 (K), D53.1 (K), D54.1 (K), D55.1 (K), D56.1 (K), D57.1 (K), D58.1 (K)
- net ROW_4: now also D59.1 (K), D60.1 (K), D61.1 (K), D62.1 (K), D63.1 (K), D64.1 (K), D65.1 (K), D66.1 (K), D67.1 (K), D68.1 (K)
- new net: D36.2 (A), SW36.2
- new net: D68.2 (A), SW68.2
- new net: D63.2 (A), SW63.2
- new net: D7.2 (A), SW7.2
- new net: D52.2 (A), SW52.2
- new net: D24.2 (A), SW24.2
- new net: D57.2 (A), SW57.2
- new net: D5.2 (A), SW5.2
- new net: D27.2 (A), SW27.2
- new net: D4.2 (A), SW4.2
- new net: D43.2 (A), SW43.2
- new net: D11.2 (A), SW11.2
- new net: D40.2 (A), SW40.2
- new net: D21.2 (A), SW21.2
- new net: D20.2 (A), SW20.2
- new net: D34.2 (A), SW34.2
- new net: D10.2 (A), SW10.2
- new net: D16.2 (A), SW16.2
- new net: D55.2 (A), SW55.2
- new net: D25.2 (A), SW25.2
- new net: D17.2 (A), SW17.2
- new net: D42.2 (A), SW42.2
- new net: D13.2 (A), SW13.2
- new net: D60.2 (A), SW60.2
- new net: D44.2 (A), SW44.2
- new net: D58.2 (A), SW58.2
- new net: D49.2 (A), SW49.2
- new net: D47.2 (A), SW47.2
- new net: D41.2 (A), SW41.2
- new net: D35.2 (A), SW35.2
- new net: D62.2 (A), SW62.2
- new net: D56.2 (A), SW56.2
- new net: D23.2 (A), SW23.2
- new net: D26.2 (A), SW26.2
- new net: D61.2 (A), SW61.2
- new net: D37.2 (A), SW37.2
- new net: D14.2 (A), SW14.2
- new net: D9.2 (A), SW9.2
- new net: D3.2 (A), SW3.2
- new net: D66.2 (A), SW66.2
- new net: D8.2 (A), SW8.2
- new net: D31.2 (A), SW31.2
- new net: D32.2 (A), SW32.2
- new net: D38.2 (A), SW38.2
- new net: D67.2 (A), SW67.2
- new net: D50.2 (A), SW50.2
- new net: D39.2 (A), SW39.2
- new net: D59.2 (A), SW59.2
- new net: D65.2 (A), SW65.2
- new net: D45.2 (A), SW45.2
- new net: D54.2 (A), SW54.2
- new net: D53.2 (A), SW53.2
- new net: D28.2 (A), SW28.2
- new net: D12.2 (A), SW12.2
- new net: D15.2 (A), SW15.2
- new net: D1.2 (A), SW1.2
- new net: D33.2 (A), SW33.2
- new net: D22.2 (A), SW22.2
- new net: D18.2 (A), SW18.2
- new net: D2.2 (A), SW2.2
- new net: D6.2 (A), SW6.2
- new net: D19.2 (A), SW19.2
- new net: D48.2 (A), SW48.2
- new net: D29.2 (A), SW29.2
- new net: D30.2 (A), SW30.2
- new net: D51.2 (A), SW51.2
- new net: D46.2 (A), SW46.2
- new net: D64.2 (A), SW64.2

Commit message: 65% PCB layout!
Parts:
- added R14, R15, R16: 10k, Resistor_SMD:R_0402_1005Metric, symbol Device:R_Small
- added SW69: EC11E15244G1, Rotary_Encoder:RotaryEncoder_Alps_EC11E_Vertical_H20mm, symbol Device:RotaryEncoder_Switch
- D1, D10, D11, D12, D13, D14, D15, D16, D17, D18, D19, D2, D20, D21, D22, D23, D24, D25, D26, D27, D28, D29, D3, D30, D31, D32, D33, D34, D35, D36, D37, D38, D39, D4, D40, D41, D42, D43, D44, D45, D46, D47, D48, D49, D5, D50, D51, D52, D53, D54, D55, D56, D57, D58, D59, D6, D60, D61, D62, D63, D64, D65, D66, D67, D68, D7, D8, D9: footprint (none) -> Diode_SMD:D_SOD-323; LCSC (none) -> C2128
- SW1, SW10, SW11, SW12, SW13, SW15, SW17, SW18, SW19, SW2, SW20, SW21, SW22, SW23, SW24, SW25, SW26, SW27, SW28, SW3, SW30, SW32, SW33, SW34, SW35, SW36, SW37, SW38, SW39, SW4, SW40, SW41, SW42, SW44, SW46, SW47, SW48, SW49, SW5, SW50, SW51, SW52, SW53, SW54, SW55, SW57, SW58, SW6, SW63, SW64, SW65, SW66, SW67, SW68, SW7, SW8, SW9: footprint (none) -> Keyboard_Switch:SW_Cherry_MX1A_1.00u_PCB
- SW14: footprint (none) -> Keyboard_Switch:SW_Cherry_MX1A_2.00u_PCB
- SW16, SW29: footprint (none) -> Keyboard_Switch:SW_Cherry_MX1A_1.50u_PCB
- SW31, SW56: footprint (none) -> Keyboard_Switch:SW_Cherry_MX1A_1.75u_PCB
- SW43, SW45: footprint (none) -> Keyboard_Switch:SW_Cherry_MX1A_2.25u_PCB
- SW59, SW60, SW61: footprint (none) -> Keyboard_Switch:SW_Cherry_MX1A_1.25u_PCB
- SW62: footprint (none) -> Keyboard_Switch:SW_Cherry_MX1A_6.25u_PCB
Connections:
- new net +3V3: R14.1, R15.1, R16.1
- new net GND: SW69.C, SW69.S2
- new net ROT_A: R15.2, SW69.A
- new net ROT_B: R16.2, SW69.B
- new net ROT_SW: R14.2, SW69.S1

Commit message: Layout Progress
Layout is finished except for the buck converter
Parts:
- SW69: footprint Rotary_Encoder:RotaryEncoder_Alps_EC11E_Vertical_H20mm -> Rotary_Encoder:RotaryEncoder_Alps_EC11E-Switch_Vertical_H20mm
Changed lines of the file:
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@@
 			)
 		)
-		(property "Footprint" "Rotary_Encoder:RotaryEncoder_Alps_EC11E_Vertical_H20mm"
+		(property "Footprint" "Rotary_Encoder:RotaryEncoder_Alps_EC11E-Switch_Vertical_H20mm"
 			(at 224.79 86.106 0)
 			(effects
