File: Keyboard_PCB/Keyboard_PCB.kicad_pcb (KiCad board)
At the start: 2 copper layers, 0 parts

Commit message: Schematic V1
Parts:
- added U1: STM32H7B0VBTx, Package_QFP:LQFP-100_14x14mm_P0.5mm, F.Cu at (150.3, 149.8)

Commit message: 65% PCB layout!
Parts:
- added C1: 1u, Capacitor_SMD:C_0402_1005Metric, B.Cu at (83.4, 225.1)
- added C10: 12p, Capacitor_SMD:C_0402_1005Metric, B.Cu at (80.6, 233.0)
- added C11: 12p, Capacitor_SMD:C_0402_1005Metric, B.Cu at (77.7, 225.1)
- added C12: 12p, Capacitor_SMD:C_0402_1005Metric, B.Cu at (77.7, 227.1)
- added C13: 12p, Capacitor_SMD:C_0402_1005Metric, B.Cu at (77.7, 229.0)
- added C14: 100n, Capacitor_SMD:C_0402_1005Metric, B.Cu at (75.6, 183.8)
- added C15: 10u, Capacitor_SMD:C_1206_3216Metric, B.Cu at (82.0, 200.4)
- added C16: 10u, Capacitor_SMD:C_1206_3216Metric, B.Cu at (82.0, 203.8)
- added C17: 100n, Capacitor_SMD:C_1206_3216Metric, B.Cu at (82.0, 207.1)
- added C18: 22u, Capacitor_SMD:C_1206_3216Metric, B.Cu at (82.0, 210.5)
- added C19: 22u, Capacitor_SMD:C_1206_3216Metric, B.Cu at (82.0, 213.8)
- added C2: 10n, Capacitor_SMD:C_0402_1005Metric, B.Cu at (83.4, 227.1)
- added C20: 4u7, Capacitor_SMD:C_0402_1005Metric, B.Cu at (75.6, 185.8)
- added C3: 4u7, Capacitor_SMD:C_0402_1005Metric, B.Cu at (83.4, 229.0)
- added C4: 100n, Capacitor_SMD:C_0402_1005Metric, B.Cu at (83.4, 231.0)
- added C5: 100n, Capacitor_SMD:C_0402_1005Metric, B.Cu at (83.4, 233.0)
- added C6: 100n, Capacitor_SMD:C_0402_1005Metric, B.Cu at (80.6, 225.1)
- added C7: 100n, Capacitor_SMD:C_0402_1005Metric, B.Cu at (80.6, 227.1)
- added C8: 100n, Capacitor_SMD:C_0402_1005Metric, B.Cu at (80.6, 229.0)
- added C9: 100n, Capacitor_SMD:C_0402_1005Metric, B.Cu at (80.6, 231.0)
- added D1: D_Small, Diode_SMD:D_SOD-323, B.Cu at (312.5, 251.8)
- added D10: D_Small, Diode_SMD:D_SOD-323, B.Cu at (312.5, 278.3)
- added D11: D_Small, Diode_SMD:D_SOD-323, B.Cu at (308.2, 251.8)
- added D12: D_Small, Diode_SMD:D_SOD-323, B.Cu at (308.2, 254.7)
- added D13: D_Small, Diode_SMD:D_SOD-323, B.Cu at (308.2, 257.7)
- added D14: D_Small, Diode_SMD:D_SOD-323, B.Cu at (308.2, 260.6)
- added D15: D_Small, Diode_SMD:D_SOD-323, B.Cu at (308.2, 263.6)
- added D16: D_Small, Diode_SMD:D_SOD-323, B.Cu at (308.2, 266.5)
- added D17: D_Small, Diode_SMD:D_SOD-323, B.Cu at (308.2, 269.5)
- added D18: D_Small, Diode_SMD:D_SOD-323, B.Cu at (308.2, 272.4)
- added D19: D_Small, Diode_SMD:D_SOD-323, B.Cu at (308.2, 275.4)
- added D2: D_Small, Diode_SMD:D_SOD-323, B.Cu at (312.5, 254.7)
- added D20: D_Small, Diode_SMD:D_SOD-323, B.Cu at (308.2, 278.3)
- added D21: D_Small, Diode_SMD:D_SOD-323, B.Cu at (303.9, 251.8)
- added D22: D_Small, Diode_SMD:D_SOD-323, B.Cu at (303.9, 254.7)
- added D23: D_Small, Diode_SMD:D_SOD-323, B.Cu at (303.9, 257.7)
- added D24: D_Small, Diode_SMD:D_SOD-323, B.Cu at (303.9, 260.6)
- added D25: D_Small, Diode_SMD:D_SOD-323, B.Cu at (303.9, 263.6)
- added D26: D_Small, Diode_SMD:D_SOD-323, B.Cu at (303.9, 266.5)
- added D27: D_Small, Diode_SMD:D_SOD-323, B.Cu at (303.9, 269.5)
- added D28: D_Small, Diode_SMD:D_SOD-323, B.Cu at (303.9, 272.4)
- added D29: D_Small, Diode_SMD:D_SOD-323, B.Cu at (303.9, 275.4)
- added D3: D_Small, Diode_SMD:D_SOD-323, B.Cu at (312.5, 257.7)
- added D30: D_Small, Diode_SMD:D_SOD-323, B.Cu at (303.9, 278.3)
- added D31: D_Small, Diode_SMD:D_SOD-323, B.Cu at (299.7, 251.8)
- added D32: D_Small, Diode_SMD:D_SOD-323, B.Cu at (299.7, 254.7)
- added D33: D_Small, Diode_SMD:D_SOD-323, B.Cu at (299.7, 257.7)
- added D34: D_Small, Diode_SMD:D_SOD-323, B.Cu at (299.7, 260.6)
- added D35: D_Small, Diode_SMD:D_SOD-323, B.Cu at (299.7, 263.6)
- added D36: D_Small, Diode_SMD:D_SOD-323, B.Cu at (299.7, 266.5)
- added D37: D_Small, Diode_SMD:D_SOD-323, B.Cu at (299.7, 269.5)
- added D38: D_Small, Diode_SMD:D_SOD-323, B.Cu at (299.7, 272.4)
- added D39: D_Small, Diode_SMD:D_SOD-323, B.Cu at (299.7, 275.4)
- added D4: D_Small, Diode_SMD:D_SOD-323, B.Cu at (312.5, 260.6)
- added D40: D_Small, Diode_SMD:D_SOD-323, B.Cu at (299.7, 278.3)
- added D41: D_Small, Diode_SMD:D_SOD-323, B.Cu at (295.4, 251.8)
- added D42: D_Small, Diode_SMD:D_SOD-323, B.Cu at (295.4, 254.7)
- added D43: D_Small, Diode_SMD:D_SOD-323, B.Cu at (295.4, 257.7)
- added D44: D_Small, Diode_SMD:D_SOD-323, B.Cu at (295.4, 260.6)
- added D45: D_Small, Diode_SMD:D_SOD-323, B.Cu at (295.4, 263.6)
- added D46: D_Small, Diode_SMD:D_SOD-323, B.Cu at (295.4, 266.5)
- added D47: D_Small, Diode_SMD:D_SOD-323, B.Cu at (295.4, 269.5)
- added D48: D_Small, Diode_SMD:D_SOD-323, B.Cu at (295.4, 272.4)
- added D49: D_Small, Diode_SMD:D_SOD-323, B.Cu at (295.4, 275.4)
- added D5: D_Small, Diode_SMD:D_SOD-323, B.Cu at (312.5, 263.6)
- added D50: D_Small, Diode_SMD:D_SOD-323, B.Cu at (295.4, 278.3)
- added D51: D_Small, Diode_SMD:D_SOD-323, B.Cu at (291.1, 251.8)
- added D52: D_Small, Diode_SMD:D_SOD-323, B.Cu at (291.1, 254.7)
- added D53: D_Small, Diode_SMD:D_SOD-323, B.Cu at (291.1, 257.7)
- added D54: D_Small, Diode_SMD:D_SOD-323, B.Cu at (291.1, 260.6)
- added D55: D_Small, Diode_SMD:D_SOD-323, B.Cu at (291.1, 263.6)
- added D56: D_Small, Diode_SMD:D_SOD-323, B.Cu at (291.1, 266.5)
- added D57: D_Small, Diode_SMD:D_SOD-323, B.Cu at (291.1, 269.5)
- added D58: D_Small, Diode_SMD:D_SOD-323, B.Cu at (291.1, 272.4)
- added D59: D_Small, Diode_SMD:D_SOD-323, B.Cu at (291.1, 275.4)
- added D6: D_Small, Diode_SMD:D_SOD-323, B.Cu at (312.5, 266.5)
- added D60: D_Small, Diode_SMD:D_SOD-323, B.Cu at (291.1, 278.3)
- added D61: D_Small, Diode_SMD:D_SOD-323, B.Cu at (286.8, 251.8)
- added D62: D_Small, Diode_SMD:D_SOD-323, B.Cu at (286.8, 254.7)
- added D63: D_Small, Diode_SMD:D_SOD-323, B.Cu at (286.8, 257.7)
- added D64: D_Small, Diode_SMD:D_SOD-323, B.Cu at (286.8, 260.6)
- added D65: D_Small, Diode_SMD:D_SOD-323, B.Cu at (286.8, 263.6)
- added D66: D_Small, Diode_SMD:D_SOD-323, B.Cu at (286.8, 266.5)
- added D67: D_Small, Diode_SMD:D_SOD-323, B.Cu at (286.8, 269.5)
- added D68: D_Small, Diode_SMD:D_SOD-323, B.Cu at (286.8, 272.4)
- added D69: 10v, Diode_SMD:D_SOD-523, B.Cu at (72.5, 204.6)
- added D7: D_Small, Diode_SMD:D_SOD-323, B.Cu at (312.5, 269.5)
- added D8: D_Small, Diode_SMD:D_SOD-323, B.Cu at (312.5, 272.4)
- added D9: D_Small, Diode_SMD:D_SOD-323, B.Cu at (312.5, 275.4)
- added FB1: 600Ω@100MHz, Inductor_SMD:L_0805_2012Metric, B.Cu at (76.9, 214.0)
- added FL1: TDK ACM2012-900, ACM2012_900_2P_T002:ACM2012_TDK, B.Cu at (76.8, 247.8)
- added J1: USB-C 16P, Connector_USB:USB_C_Receptacle_HCTL_HC-TYPE-C-16P-01A, B.Cu at (79.0, 241.4)
- added L1: 10u, Inductor_SMD:L_0603_1608Metric, B.Cu at (73.9, 218.8)
- added L2: 2u2, Inductor_SMD:L_Changjiang_FNR3015S, B.Cu at (76.9, 210.3)
- added Q1: AO3401A, Package_TO_SOT_SMD:SOT-23, B.Cu at (76.8, 205.8)
- added Q2: S8050, Package_TO_SOT_SMD:SOT-23, B.Cu at (79.5, 185.2)
- added R1: 5k1, Resistor_SMD:R_0603_1608Metric, B.Cu at (72.7, 247.3)
- added R10: 2k2, Resistor_SMD:R_0402_1005Metric, B.Cu at (83.4, 189.8)
- added R11: 2k2, Resistor_SMD:R_0402_1005Metric, B.Cu at (83.4, 191.8)
- added R12: 22, Resistor_SMD:R_0402_1005Metric, B.Cu at (83.4, 193.7)
- added R13: 22, Resistor_SMD:R_0402_1005Metric, B.Cu at (83.4, 195.7)
- added R14: 10k, Resistor_SMD:R_0402_1005Metric, B.Cu at (283.2, 266.0)
- added R15: 10k, Resistor_SMD:R_0402_1005Metric, B.Cu at (283.2, 268.0)
- added R16: 10k, Resistor_SMD:R_0402_1005Metric, B.Cu at (283.2, 270.0)
- added R2: 47, Resistor_SMD:R_0402_1005Metric, B.Cu at (74.4, 221.0)
- added R3: 47, Resistor_SMD:R_0402_1005Metric, B.Cu at (74.4, 223.0)
- added R4: 10k, Resistor_SMD:R_0603_1608Metric, B.Cu at (72.6, 209.2)
- added R5: 33k2, Resistor_SMD:R_0603_1608Metric, B.Cu at (72.6, 211.7)
- added R6: 10k, Resistor_SMD:R_0603_1608Metric, B.Cu at (72.6, 214.2)
- added R7: 8r2, Resistor_SMD:R_0402_1005Metric, B.Cu at (83.4, 183.8)
- added R8: 10k, Resistor_SMD:R_0402_1005Metric, B.Cu at (83.4, 185.8)
- added R9: 1k, Resistor_SMD:R_0402_1005Metric, B.Cu at (83.4, 187.8)
- added SW1: ESC, Keyboard_Switch:SW_Cherry_MX1A_1.00u_PCB, F.Cu at (38.1, 38.1)
- added SW10: 9, Keyboard_Switch:SW_Cherry_MX1A_1.00u_PCB, F.Cu at (209.6, 38.1)
- added SW11: 0, Keyboard_Switch:SW_Cherry_MX1A_1.00u_PCB, F.Cu at (228.6, 38.1)
- added SW12: -, Keyboard_Switch:SW_Cherry_MX1A_1.00u_PCB, F.Cu at (247.7, 38.1)
- added SW13: =, Keyboard_Switch:SW_Cherry_MX1A_1.00u_PCB, F.Cu at (266.7, 38.1)
- added SW14: <-, Keyboard_Switch:SW_Cherry_MX1A_2.00u_PCB, F.Cu at (295.3, 38.1)
- added SW15: DEL, Keyboard_Switch:SW_Cherry_MX1A_1.00u_PCB, F.Cu at (323.9, 38.1)
- added SW16: TAB, Keyboard_Switch:SW_Cherry_MX1A_1.50u_PCB, F.Cu at (42.9, 57.1)
- added SW17: Q, Keyboard_Switch:SW_Cherry_MX1A_1.00u_PCB, F.Cu at (66.7, 57.1)
- added SW18: W, Keyboard_Switch:SW_Cherry_MX1A_1.00u_PCB, F.Cu at (85.7, 57.1)
- added SW19: E, Keyboard_Switch:SW_Cherry_MX1A_1.00u_PCB, F.Cu at (104.8, 57.1)
- added SW2: 1, Keyboard_Switch:SW_Cherry_MX1A_1.00u_PCB, F.Cu at (57.1, 38.1)
- added SW20: R, Keyboard_Switch:SW_Cherry_MX1A_1.00u_PCB, F.Cu at (123.8, 57.1)
- added SW21: T, Keyboard_Switch:SW_Cherry_MX1A_1.00u_PCB, F.Cu at (142.9, 57.1)
- added SW22: Y, Keyboard_Switch:SW_Cherry_MX1A_1.00u_PCB, F.Cu at (161.9, 57.1)
- added SW23: U, Keyboard_Switch:SW_Cherry_MX1A_1.00u_PCB, F.Cu at (181.0, 57.1)
- added SW24: I, Keyboard_Switch:SW_Cherry_MX1A_1.00u_PCB, F.Cu at (200.0, 57.1)
- added SW25: O, Keyboard_Switch:SW_Cherry_MX1A_1.00u_PCB, F.Cu at (219.1, 57.1)
- added SW26: P, Keyboard_Switch:SW_Cherry_MX1A_1.00u_PCB, F.Cu at (238.1, 57.1)
- added SW27: [, Keyboard_Switch:SW_Cherry_MX1A_1.00u_PCB, F.Cu at (257.2, 57.1)
- added SW28: ], Keyboard_Switch:SW_Cherry_MX1A_1.00u_PCB, F.Cu at (276.2, 57.1)
- added SW29: \, Keyboard_Switch:SW_Cherry_MX1A_1.50u_PCB, F.Cu at (300.0, 57.1)
- added SW3: 2, Keyboard_Switch:SW_Cherry_MX1A_1.00u_PCB, F.Cu at (76.2, 38.1)
- added SW30: HOME, Keyboard_Switch:SW_Cherry_MX1A_1.00u_PCB, F.Cu at (323.9, 57.1)
- added SW31: CAPS, Keyboard_Switch:SW_Cherry_MX1A_1.75u_PCB, F.Cu at (45.2, 76.2)
- added SW32: A, Keyboard_Switch:SW_Cherry_MX1A_1.00u_PCB, F.Cu at (71.4, 76.2)
- added SW33: S, Keyboard_Switch:SW_Cherry_MX1A_1.00u_PCB, F.Cu at (90.5, 76.2)
- added SW34: D, Keyboard_Switch:SW_Cherry_MX1A_1.00u_PCB, F.Cu at (109.5, 76.2)
- added SW35: F, Keyboard_Switch:SW_Cherry_MX1A_1.00u_PCB, F.Cu at (128.6, 76.2)
- added SW36: G, Keyboard_Switch:SW_Cherry_MX1A_1.00u_PCB, F.Cu at (147.6, 76.2)
- added SW37: H, Keyboard_Switch:SW_Cherry_MX1A_1.00u_PCB, F.Cu at (166.7, 76.2)
- added SW38: J, Keyboard_Switch:SW_Cherry_MX1A_1.00u_PCB, F.Cu at (185.7, 76.2)
- added SW39: K, Keyboard_Switch:SW_Cherry_MX1A_1.00u_PCB, F.Cu at (204.8, 76.2)
- added SW4: 3, Keyboard_Switch:SW_Cherry_MX1A_1.00u_PCB, F.Cu at (95.2, 38.1)
- added SW40: L, Keyboard_Switch:SW_Cherry_MX1A_1.00u_PCB, F.Cu at (223.8, 76.2)
- added SW41: ;, Keyboard_Switch:SW_Cherry_MX1A_1.00u_PCB, F.Cu at (242.9, 76.2)
- added SW42: ', Keyboard_Switch:SW_Cherry_MX1A_1.00u_PCB, F.Cu at (261.9, 76.2)
- added SW43: ENTER, Keyboard_Switch:SW_Cherry_MX1A_2.25u_PCB, F.Cu at (292.9, 76.2)
- added SW44: PG_U, Keyboard_Switch:SW_Cherry_MX1A_1.00u_PCB, F.Cu at (323.9, 76.2)
- added SW45: SHIFT, Keyboard_Switch:SW_Cherry_MX1A_2.25u_PCB, F.Cu at (50.0, 95.2)
- added SW46: Z, Keyboard_Switch:SW_Cherry_MX1A_1.00u_PCB, F.Cu at (81.0, 95.2)
- added SW47: X, Keyboard_Switch:SW_Cherry_MX1A_1.00u_PCB, F.Cu at (100.0, 95.2)
- added SW48: C, Keyboard_Switch:SW_Cherry_MX1A_1.00u_PCB, F.Cu at (119.1, 95.2)
- added SW49: V, Keyboard_Switch:SW_Cherry_MX1A_1.00u_PCB, F.Cu at (138.1, 95.2)
- added SW5: 4, Keyboard_Switch:SW_Cherry_MX1A_1.00u_PCB, F.Cu at (114.3, 38.1)
- added SW50: B, Keyboard_Switch:SW_Cherry_MX1A_1.00u_PCB, F.Cu at (157.2, 95.2)
- added SW51: N, Keyboard_Switch:SW_Cherry_MX1A_1.00u_PCB, F.Cu at (176.2, 95.2)
- added SW52: M, Keyboard_Switch:SW_Cherry_MX1A_1.00u_PCB, F.Cu at (195.3, 95.2)
- added SW53: ,, Keyboard_Switch:SW_Cherry_MX1A_1.00u_PCB, F.Cu at (214.3, 95.2)
- added SW54: ., Keyboard_Switch:SW_Cherry_MX1A_1.00u_PCB, F.Cu at (233.4, 95.2)
- added SW55: /, Keyboard_Switch:SW_Cherry_MX1A_1.00u_PCB, F.Cu at (252.4, 95.2)
- added SW56: SHIFT, Keyboard_Switch:SW_Cherry_MX1A_1.75u_PCB, F.Cu at (278.6, 95.2)
- added SW57: UP, Keyboard_Switch:SW_Cherry_MX1A_1.00u_PCB, F.Cu at (304.8, 95.2)
- added SW58: PG_D, Keyboard_Switch:SW_Cherry_MX1A_1.00u_PCB, F.Cu at (323.9, 95.2)
- added SW59: CTRL, Keyboard_Switch:SW_Cherry_MX1A_1.25u_PCB, F.Cu at (40.5, 114.3)
- added SW6: 5, Keyboard_Switch:SW_Cherry_MX1A_1.00u_PCB, F.Cu at (133.3, 38.1)
- added SW60: CODE, Keyboard_Switch:SW_Cherry_MX1A_1.25u_PCB, F.Cu at (64.3, 114.3)
- added SW61: ALT, Keyboard_Switch:SW_Cherry_MX1A_1.25u_PCB, F.Cu at (88.1, 114.3)
- added SW62: SPACE, Keyboard_Switch:SW_Cherry_MX1A_6.25u_PCB, F.Cu at (159.5, 114.3)
- added SW63: ALT, Keyboard_Switch:SW_Cherry_MX1A_1.00u_PCB, F.Cu at (228.6, 114.3)
- added SW64: CODE, Keyboard_Switch:SW_Cherry_MX1A_1.00u_PCB, F.Cu at (247.7, 114.3)
- added SW65: CTRL, Keyboard_Switch:SW_Cherry_MX1A_1.00u_PCB, F.Cu at (266.7, 114.3)
- added SW66: LEFT, Keyboard_Switch:SW_Cherry_MX1A_1.00u_PCB, F.Cu at (285.8, 114.3)
- added SW67: DOWN, Keyboard_Switch:SW_Cherry_MX1A_1.00u_PCB, F.Cu at (304.8, 114.3)
- added SW68: RIGHT, Keyboard_Switch:SW_Cherry_MX1A_1.00u_PCB, F.Cu at (323.9, 114.3)
- added SW69: EC11E15244G1, Rotary_Encoder:RotaryEncoder_Alps_EC11E_Vertical_H20mm, B.Cu at (282.9, 255.2)
- added SW7: 6, Keyboard_Switch:SW_Cherry_MX1A_1.00u_PCB, F.Cu at (152.4, 38.1)
- added SW8: 7, Keyboard_Switch:SW_Cherry_MX1A_1.00u_PCB, F.Cu at (171.4, 38.1)
- added SW9: 8, Keyboard_Switch:SW_Cherry_MX1A_1.00u_PCB, F.Cu at (190.5, 38.1)
- added U2: USBLC6-2SC6, Package_TO_SOT_SMD:SOT-23-6, B.Cu at (82.3, 248.5)
- added U3: ~, Package_TO_SOT_SMD:SOT-23-6, B.Cu at (76.6, 201.1)
- added U4: ~, Package_SO:PowerIntegrations_SO-8, B.Cu at (80.4, 220.9)
- added U5: ~, Custom:FPC_30_soldered, B.Cu at (76.7, 182.1)
- added Y1: 25MHz, Crystal:Crystal_SMD_3225-4Pin_3.2x2.5mm, B.Cu at (73.6, 226.3)
- added Y2: 32.768 KHz, Crystal:Crystal_SMD_3215-2Pin_3.2x1.5mm, B.Cu at (73.7, 230.2)
- U1: moved to B.Cu
- moved U1 102.9 mm to (178.3, 248.8), turned to 180 degrees
Connections:
- U1 pad 10: Net-(U1-VSS-Pad10) -> GND
- U1 pad 100: unconnected-(U1-VDD-Pad100) -> +3V3
- U1 pad 11: unconnected-(U1-VDD-Pad11) -> +3V3
- U1 pad 19: unconnected-(U1-VSSA-Pad19) -> GND
- U1 pad 21: unconnected-(U1-VDDA-Pad21) -> +3.3VA
- U1 pad 22: unconnected-(U1-PA0-Pad22) -> /TIM_CH1
- U1 pad 23: unconnected-(U1-PA1-Pad23) -> /TIM_CH2
- U1 pad 24: unconnected-(U1-PA2-Pad24) -> /ROT_SW
- U1 pad 26: Net-(U1-VSS-Pad10) -> GND
- U1 pad 27: unconnected-(U1-VDD-Pad27) -> +3V3
- U1 pad 46: unconnected-(U1-PB10-Pad46) -> /LCD_CMD
- U1 pad 47: unconnected-(U1-PB11-Pad47) -> /LCD_NRST
- U1 pad 49: Net-(U1-VSS-Pad10) -> GND
- U1 pad 50: unconnected-(U1-VDD-Pad50) -> +3V3
- U1 pad 53: unconnected-(U1-PB14-Pad53) -> /LCD_BL
- U1 pad 6: unconnected-(U1-VBAT-Pad6) -> +3V3
- U1 pad 74: Net-(U1-VSS-Pad10) -> GND
- U1 pad 75: unconnected-(U1-VDD-Pad75) -> +3V3
- U1 pad 99: Net-(U1-VSS-Pad10) -> GND

Commit message: Rough Layout
Parts:
- moved D1 209.6 mm to (120.4, 168.0), turned to 90 degrees
- moved D16 205.9 mm to (118.7, 186.1)
- moved R2 201.9 mm to (275.8, 235.5)
- moved R3 201.9 mm to (275.8, 237.5)
- moved L1 201.9 mm to (275.2, 233.2)
- moved C1 201.5 mm to (284.6, 236.1)
- moved C10 201.5 mm to (281.7, 244.0)
- moved C11 201.5 mm to (278.9, 236.1)
- moved C12 201.5 mm to (278.9, 238.1)
- moved C13 201.5 mm to (278.9, 240.1)
- moved C2 201.5 mm to (284.6, 238.1)
- moved C3 201.5 mm to (284.6, 240.1)
- moved C4 201.5 mm to (284.6, 242.0)
- moved C5 201.5 mm to (284.6, 244.0)
- moved C6 201.5 mm to (281.7, 236.1)
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Connections:
- SW69 pad : (no net) -> GND
Routing:
- added copper zone on In2.Cu, net +3V3
- added copper zone on In1.Cu, net GND
Other:
- board outline added: 304 x 92.2 mm
- copper layers 2 -> 4

Commit message: Layout Progress
Layout is finished except for the buck converter
Parts:
- added C21: 2u2, Capacitor_SMD:C_0402_1005Metric, B.Cu at (251.7, 235.0)
- added C22: 2u2, Capacitor_SMD:C_0402_1005Metric, B.Cu at (259.5, 221.4)
- added J2: JTAG, Connector_PinHeader_2.00mm:PinHeader_2x04_P2.00mm_Vertical, F.Cu at (295.4, 235.0)
- added JP1: SolderJumper_2_Open, Jumper:SolderJumper-2_P1.3mm_Open_TrianglePad1.0x1.5mm, B.Cu at (274.5, 224.6)
- added JP2: SolderJumper_2_Open, Jumper:SolderJumper-2_P1.3mm_Open_TrianglePad1.0x1.5mm, B.Cu at (277.0, 224.5)
- SW69: footprint Rotary_Encoder:RotaryEncoder_Alps_EC11E_Vertical_H20mm -> Rotary_Encoder:RotaryEncoder_Alps_EC11E-Switch_Vertical_H20mm
- moved C9 31.9 mm to (251.2, 233.0), turned to -135 degrees
- moved C8 27.9 mm to (261.5, 220.8), turned to 135 degrees
- moved C7 22.8 mm to (259.4, 242.8), turned to -45 degrees
- moved C5 18.8 mm to (273.2, 229.0), turned to 135 degrees
- moved C2 18.4 mm to (267.2, 244.0), turned to -45 degrees
- moved C1 18.0 mm to (268.0, 243.2), turned to -45 degrees
- moved C3 15.9 mm to (274.0, 228.2), turned to 135 degrees
- moved L1 13.9 mm to (265.4, 243.0), turned to -135 degrees
- moved C4 13.4 mm to (273.6, 234.4), turned to 45 degrees
- moved C11 12.7 mm to (267.1, 241.0), turned to -135 degrees
- moved C14 12.0 mm to (206.7, 240.6), turned to 0 degrees
- moved C6 11.7 mm to (270.2, 238.0), turned to 45 degrees
- moved R13 11.3 mm to (205.0, 239.6)
- moved R7 9.99 mm to (196.5, 240.2), turned to -90 degrees
- moved C20 9.95 mm to (206.7, 239.4), turned to 0 degrees
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Connections:
- U1 pad 48: unconnected-(U1-VCAP-Pad48) -> Net-(C21-Pad1)
- U1 pad 73: unconnected-(U1-VCAP-Pad73) -> Net-(C22-Pad1)
- U1 pad 94: /BOOT_0 -> /BOOT0
Routing:
- net /ROW_0: track 0.00 -> 371.7 mm, vias 0 -> 15
- net /ROW_1: track 0.00 -> 350.7 mm, vias 0 -> 15
- net /ROW_2: track 0.00 -> 324.0 mm, vias 0 -> 14
- net /ROW_4: track 0.00 -> 309.9 mm, vias 0 -> 13
- net /ROW_3: track 0.00 -> 301.2 mm, vias 0 -> 15
- net /COL_14: track 0.00 -> 229.7 mm, vias 0 -> 1
- net /COL_0: track 0.00 -> 223.7 mm, vias 0 -> 1
- net /COL_13: track 0.00 -> 220.7 mm, vias 0 -> 1
- net /COL_11: track 0.00 -> 209.0 mm, vias 0 -> 1
- net /COL_1: track 0.00 -> 206.4 mm, vias 0 -> 1
- net /COL_12: track 0.00 -> 192.0 mm, vias 0 -> 2
- net /COL_10: track 0.00 -> 189.0 mm, vias 0 -> 1
- net /COL_2: track 0.00 -> 187.4 mm, vias 0 -> 1
- net /USB_DN: track 0.00 -> 184.6 mm, vias 0 -> 2
- net /USB_DP: track 0.00 -> 184.5 mm, vias 0 -> 2
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
Commit message: Layout Progress
Parts:
- removed C15, C16: 10u, Capacitor_SMD:C_1206_3216Metric
- removed C17: 100n, Capacitor_SMD:C_1206_3216Metric
- removed C18, C19: 22u, Capacitor_SMD:C_1206_3216Metric
- removed D69: 10v, Diode_SMD:D_SOD-523
- removed FB1: 600Ω@100MHz, Inductor_SMD:L_0805_2012Metric
- removed L2: 2u2, Inductor_SMD:L_Changjiang_FNR3015S
- removed Q1: AO3401A, Package_TO_SOT_SMD:SOT-23
- removed R4, R6: 10k, Resistor_SMD:R_0603_1608Metric
- removed R5: 33k2, Resistor_SMD:R_0603_1608Metric
- removed U3: ~, Package_TO_SOT_SMD:SOT-23-6
- moved R15 13.3 mm to (226.4, 228.0), turned to -90 degrees
- moved R14 7.69 mm to (226.4, 243.6), turned to -90 degrees
- moved R16 3.03 mm to (226.4, 230.6), turned to 90 degrees
- moved SW69 1.72 mm to (215.9, 228.6)
Routing:
- net +5V: track 17.6 -> 104.2 mm
- net /SPI_NCS: track 55.6 -> 58.9 mm
- net /SPI_CLK: track 60.9 -> 64.1 mm
- net /SPI_MOSI: track 62.7 -> 66.0 mm
- net /LCD_BL: track 63.2 -> 65.5 mm
- net +3V3: track 48.9 -> 47.1 mm
- net /LCD_NRST: track 56.7 -> 58.0 mm
- net /LCD_CMD: track 58.3 -> 59.5 mm
- net /ROT_SW: track 47.4 -> 46.4 mm
- net /TIM_CH2: track 50.5 -> 49.8 mm
- net /TIM_CH1: track 56.4 -> 56.0 mm, vias 1 -> 2

Commit message: Added TODO's
Other:
- board text added: "TODO: MOUNTING HOLES TODO: NEW BUCK CONVERTER"
Changed lines of the file:
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@@
 		(layer "Edge.Cuts")
+	)
+	(gr_text "TODO: MOUNTING HOLES\nTODO: NEW BUCK CONVERTER"
+		(at 211.20375 116.0425 0)
+		(layer "Cmts.User")
+		(effects
+			(font
+				(size 5.08 5.08)
+				(thickness 0.3)
+				(bold yes)
+			)
+			(justify left bottom)
+		)
 	)
 	(segment

Commit message: Layout V1
Parts:
- added C15: 10u, Capacitor_SMD:C_1206_3216Metric, B.Cu at (144.0, 163.8)
- added C16: 10u, Capacitor_SMD:C_1206_3216Metric, B.Cu at (146.6, 163.8)
- added C17: 100n, Capacitor_SMD:C_1206_3216Metric, B.Cu at (145.2, 171.4)
- added C18: 22u, Capacitor_SMD:C_1206_3216Metric, B.Cu at (153.3, 171.4)
- added C19: 22u, Capacitor_SMD:C_1206_3216Metric, B.Cu at (155.8, 171.4)
- added D69: 10v, Diode_SMD:D_SOD-523, B.Cu at (144.0, 157.4)
- added FB1: 600Ω@100MHz, Inductor_SMD:L_0805_2012Metric, B.Cu at (145.2, 160.2)
- added H1: MountingHole_Pad, MountingHole:MountingHole_2.2mm_M2_DIN965_Pad, F.Cu at (367.4, 180.8)
- added H2: MountingHole_Pad, MountingHole:MountingHole_2.2mm_M2_DIN965_Pad, F.Cu at (131.9, 180.8)
- added H3: MountingHole_Pad, MountingHole:MountingHole_2.2mm_M2_DIN965_Pad, F.Cu at (235.4, 199.8)
- added H4: MountingHole_Pad, MountingHole:MountingHole_2.2mm_M2_DIN965_Pad, F.Cu at (373.4, 237.5)
- added H5: MountingHole_Pad, MountingHole:MountingHole_2.2mm_M2_DIN965_Pad, F.Cu at (294.9, 237.5)
- added H6: MountingHole_Pad, MountingHole:MountingHole_2.2mm_M2_DIN965_Pad, F.Cu at (131.9, 237.5)
- added L2: 2u2, Inductor_SMD:L_Changjiang_FNR3015S, B.Cu at (150.0, 172.0)
- added Q1: AO3401A, Package_TO_SOT_SMD:SOT-23, B.Cu at (140.9, 157.8)
- added R4: 10k, Resistor_SMD:R_0603_1608Metric, B.Cu at (146.4, 157.6)
- added R5: 33k2, Resistor_SMD:R_0603_1608Metric, B.Cu at (149.0, 168.2)
- added R6: 10k, Resistor_SMD:R_0603_1608Metric, B.Cu at (149.0, 165.0)
- added U3: ~, Package_TO_SOT_SMD:SOT-23-6, B.Cu at (145.2, 168.2)
- moved J2 14.0 mm to (281.4, 234.8)
- moved R1 4.21 mm to (128.0, 162.7)
- moved FL1 1.33 mm to (125.1, 166.9)
- moved U2 1.33 mm to (125.2, 163.3)
- moved J1 1.28 mm to (125.2, 156.0)
- moved C14 0.20 mm to (206.7, 240.4)
- moved C20 0.10 mm to (206.7, 239.3)
- turned R13 to -90 degrees
Connections:
- net /LCD/LCD_LEDK renamed /LCD/FPC_LEDK
- net /LCD/LCD_NSS renamed /LCD/FPC_NCS
- R13 pad 2: /LCD_NRST -> /LCD/FPC_NRST
- U5 pad 5: /LCD_NRST -> /LCD/FPC_NRST
Routing:
- net +5V: track 104.2 -> 253.2 mm, vias 3 -> 5
- net GND: track 83.2 -> 117.0 mm, vias 39 -> 50
- net /Power/BUCK_EN: track 0.00 -> 19.1 mm
- net +3V3: track 47.1 -> 62.8 mm, vias 23 -> 27
- net /NRST: track 32.2 -> 18.1 mm
- net /SWDIO: track 41.8 -> 27.9 mm
- net /SWCLK: track 43.4 -> 29.6 mm
- net /Power/BUCK_SW: track 0.00 -> 10.4 mm
- net Net-(D69-A): track 0.00 -> 4.62 mm
- net Net-(D69-K): track 0.00 -> 4.40 mm
- net /Power/BUCK_FB: track 0.00 -> 4.26 mm
- net /LCD_NRST: track 58.0 -> 54.6 mm
- net /LCD/FPC_NRST: track 0.00 -> 3.41 mm
- net /Power/BUCK_BST: track 0.00 -> 2.39 mm
- net /USB_DN: track 184.6 -> 183.4 mm
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Other:
- board text removed: "TODO: MOUNTING HOLES TODO: NEW BUCK CONVERTER"
