File: Keyboard_PCB/Keyboard_PCB.kicad_pcb (KiCad board)
At the start: 4 copper layers, 42 x 62.5 mm, 101 parts, among them J1 I2C_LCD, J2 USB-C 16P, J3 LCD_MODULE, J4 FPC 30, J5 JTAG, Q1 S8050, SW1 EC11E15244G1, SW2 BTN, SW3 BTN, SW4 BTN, U1 STM32F412CGUx, U2 ISL91127IR, U3 USBLC6-2SC6, U4 ISL91127IR, U5 MCP73833, U6 MCP73833, U7 W25Q128JVS, Y1 25MHz, Y2 32.768 KHz

Commit message: Keyboard V2 outline
Parts:
- removed BT1: APP, Connector_PinHeader_2.54mm:PinHeader_1x02_P2.54mm_Vertical
- removed BT2: BKUP, Connector_PinHeader_2.54mm:PinHeader_1x02_P2.54mm_Vertical
- removed C1, C2, C9: 10n, Capacitor_SMD:C_0603_1608Metric
- removed C10, C12, C3, C4, C5, C6, C8: 100n, Capacitor_SMD:C_0603_1608Metric
- removed C11, C7: 4u7, Capacitor_SMD:C_0603_1608Metric
- removed C13: 2u2, Capacitor_SMD:C_0603_1608Metric
- removed C14, C17: 10u, Capacitor_SMD:C_0603_1608Metric
- removed C15, C16, C18, C19: 22u, Capacitor_SMD:C_0603_1608Metric
- removed C20, C21, C22, C23: 1u, Capacitor_SMD:C_0603_1608Metric
- removed C28, C29, C30, C35: 12p, Capacitor_SMD:C_0603_1608Metric
- removed D1: STATUS, LED_SMD:LED_0603_1608Metric
- removed D10, D7: STAT2, LED_SMD:LED_0603_1608Metric
- removed D11, D8: PG, LED_SMD:LED_0603_1608Metric
- removed D2: PWR, LED_SMD:LED_0603_1608Metric
- removed D3: 5v1, Diode_SMD:D_SOD-123
- removed D4, D5: BAT54C, Package_TO_SOT_SMD:SOT-23
- removed D6, D9: STAT1, LED_SMD:LED_0603_1608Metric
- removed F1: 6V/2A, Fuse:Fuse_1206_3216Metric
- removed FL1: TDK ACM2012-900, ACM2012_900_2P_T002:ACM2012_TDK
- removed H1, H2, H3, H4: MountingHole_Pad, MountingHole:MountingHole_2.2mm_M2_Pad_Via
- removed J1: I2C_LCD, Connector_PinHeader_2.54mm:PinHeader_1x04_P2.54mm_Vertical
- removed J2: USB-C 16P, Connector_USB:USB_C_Receptacle_HCTL_HC-TYPE-C-16P-01A
- removed J3: LCD_MODULE, Connector_PinHeader_2.54mm:PinHeader_2x04_P2.54mm_Vertical
- removed J4: FPC 30, Marijn_KiCad:SMD_FPC30
- removed J5: JTAG, Connector_PinHeader_2.54mm:PinHeader_1x04_P2.54mm_Vertical
- removed JP1: PWR_LED, Jumper:SolderJumper-2_P1.3mm_Open_TrianglePad1.0x1.5mm
- removed JP2: WKUP_EXTI, Jumper:SolderJumper-2_P1.3mm_Open_TrianglePad1.0x1.5mm
- removed JP3: VBAT_BYP, Jumper:SolderJumper-2_P1.3mm_Open_TrianglePad1.0x1.5mm
- removed L1: 10u, Inductor_SMD:L_0805_2012Metric
- removed L2, L3: 1u, Inductor_SMD:L_0805_2012Metric
- removed Q1: S8050, Package_TO_SOT_SMD:SOT-23
- removed R1, R12, R2, R22, R23, R26, R3, R4, R5, R6, R8, TH1, TH2: 10k, Resistor_SMD:R_0603_1608Metric
- removed R10, R11, R13, R14, R15, R9: 470, Resistor_SMD:R_0603_1608Metric
- removed R24, R27: 1k, Resistor_SMD:R_0603_1608Metric
- removed R25, R7: 5k1, Resistor_SMD:R_0603_1608Metric
- removed R28: 8R2, Resistor_SMD:R_0603_1608Metric
- removed R29, R30: 47, Resistor_SMD:R_0603_1608Metric
- removed SW1: EC11E15244G1, Rotary_Encoder:RotaryEncoder_Alps_EC11E-Switch_Vertical_H20mm
- removed SW2: BTN, Button_Switch_Keyboard:SW_Cherry_MX_1.00u_PCB
- removed SW3, SW4: BTN, Button_Switch_SMD:SW_SPST_PTS810
- removed TP1: 5V, TestPoint:TestPoint_Pad_D2.0mm
- removed TP2: 3V3, TestPoint:TestPoint_Pad_D1.5mm
- removed TP3: Vbat, TestPoint:TestPoint_Pad_D1.5mm
- removed U1: STM32F412CGUx, Package_DFN_QFN:QFN-48-1EP_7x7mm_P0.5mm_EP5.6x5.6mm
- removed U2, U4: ISL91127IR, Package_DFN_QFN:QFN-20-1EP_4x4mm_P0.5mm_EP2.7x2.7mm_ThermalVias
- removed U3: USBLC6-2SC6, Package_TO_SOT_SMD:SOT-23-6
- removed U5, U6: MCP73833, Package_DFN_QFN:DFN-10-1EP_3x3mm_P0.5mm_EP1.58x2.35mm
- removed U7: W25Q128JVS, Marijn_KiCad:SOIC-8_W25QxJVS
- removed Y1: 25MHz, Crystal:Crystal_SMD_3225-4Pin_3.2x2.5mm
- removed Y2: 32.768 KHz, Crystal:Crystal_SMD_3215-2Pin_3.2x1.5mm
Routing:
- net GND: track 86.2 -> 0.00 mm, vias 261 -> 0
- net /ENC_SW: track 52.3 -> 0.00 mm, vias 3 -> 0
- net /USB_SENS: track 50.1 -> 0.00 mm, vias 6 -> 0
- net /ENC_A: track 44.6 -> 0.00 mm, vias 2 -> 0
- net +5V: track 40.9 -> 0.00 mm, vias 11 -> 0
- net /ENC_B: track 40.4 -> 0.00 mm, vias 2 -> 0
- net /SWDIO: track 36.3 -> 0.00 mm, vias 3 -> 0
- net /LCD_NRST: track 35.9 -> 0.00 mm, vias 3 -> 0
- net /SWCLK: track 34.5 -> 0.00 mm, vias 1 -> 0
- net /LCD_DC: track 33.9 -> 0.00 mm, vias 3 -> 0
- net +3V3: track 32.6 -> 0.00 mm, vias 33 -> 0
- net /LCD_CLK: track 31.9 -> 0.00 mm, vias 2 -> 0
- net /VBAT: track 28.7 -> 0.00 mm, vias 2 -> 0
- net /LCD_NCS: track 28.7 -> 0.00 mm, vias 3 -> 0
- net /LCD_MOSI: track 28.0 -> 0.00 mm, vias 3 -> 0
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- removed copper zone on F.Cu, net +3V3
- removed copper zone on In2.Cu, net +3V3
- removed copper zone on B.Cu, net +5V
- removed copper zone on F.Cu, net +5V
- removed copper zone on F.Cu, net /BOOT0
- removed copper zone on F.Cu, net /NRST
- removed copper zone on F.Cu, net /USB_PWR/APP_BAT
- removed copper zone on F.Cu, net /USB_PWR/APP_PROG
- removed copper zone on F.Cu, net /USB_PWR/BKUP_BAT
- removed copper zone on F.Cu, net /USB_PWR/BKUP_PROG
- removed copper zone on F.Cu, net /USB_PWR/PVIN_APP
- removed copper zone on F.Cu, net /USB_PWR/PVIN_BKUP
- removed copper zone on F.Cu, net /VBAT
- removed copper zone on B.Cu, net GND
- removed copper zone on F.Cu, net GND
- removed copper zone on In1.Cu, net GND
- removed copper zone on F.Cu, net Net-(L2-Pad1)
- removed copper zone on F.Cu, net Net-(L2-Pad2)
- removed copper zone on F.Cu, net Net-(L3-Pad1)
- removed copper zone on F.Cu, net Net-(L3-Pad2)
Other:
- board size 42 x 62.5 mm -> 305 x 132 mm
- board text removed: "BT1"
- board text removed: "BT2"
- board text removed: "FPC_30"
- board text removed: "I2C_LCD"
- board text removed: "J1"
- board text removed: "J3"
- board text removed: "J5"
- board text removed: "JTAG"
- board text removed: "KB PCB V0"
- board text removed: "PWR"
- board text removed: "ROT/BTN"
- board text removed: "SPI_LCD"
- board text removed: "STAT"
- board text removed: "SW1"
- board text removed: "SW2"
- board text removed: "VBAT_BYP"
- board text removed: "WKUP/BTN"
- board text removed: "WKUP_EXTI"
