File: Keyboard_PCB/lcd.kicad_sch (KiCad schematic)
At the start: 11 parts, among them Q2 S8050

Commit message: Layout V1
Connections:
- net LCD_NRST: no longer R13.2, U5.5 (RES)
- net LCD_LEDK renamed FPC_LEDK
- net LCD_NSS renamed FPC_NCS
- new net FPC_NRST: R13.2, U5.5 (RES)
Changed lines of the file:
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@@
 		)
 	)
-	(label "LCD_NRST"
+	(label "FPC_NRST"
 		(at 209.55 54.61 180)
 		(fields_autoplaced yes)
@@
 		)
 	)
-	(label "LCD_NSS"
+	(label "FPC_NCS"
 		(at 209.55 57.15 180)
 		(fields_autoplaced yes)
@@
 		)
 	)
-	(label "LCD_NRST"
+	(label "FPC_NRST"
 		(at 148.59 66.04 0)
 		(fields_autoplaced yes)
@@
 		)
 	)
-	(label "LCD_NSS"
+	(label "FPC_NCS"
 		(at 128.27 66.04 180)
 		(fields_autoplaced yes)
@@
 		)
 	)
-	(label "LCD_LEDK"
+	(label "FPC_LEDK"
 		(at 205.74 95.25 180)
 		(fields_autoplaced yes)
@@
 		)
 	)
-	(label "LCD_LEDK"
+	(label "FPC_LEDK"
 		(at 157.48 83.82 0)
 		(fields_autoplaced yes)
