File: Keyboard_PCB/power.kicad_sch (KiCad schematic)
At the start: 0 parts

Commit message: Schematic V1
Parts:
- added C15, C16: 10u, Capacitor_SMD:C_1206_3216Metric, symbol Device:C_Small
- added C17: 100n, Capacitor_SMD:C_1206_3216Metric, symbol Device:C_Small
- added C18, C19: 22u, Capacitor_SMD:C_1206_3216Metric, symbol Device:C_Small
- added D69: 10v, Diode_SMD:D_SOD-523, symbol Device:D_Zener_Small
- added FB1: 600Ω@100MHz, symbol Device:FerriteBead_Small
- added L2: 2u2, Inductor_SMD:L_Changjiang_FNR3015S, symbol Device:L_Small
- added Q1: AO3401A, Package_TO_SOT_SMD:SOT-23, symbol Transistor_FET:AO3401A
- added R4, R6: 10k, Resistor_SMD:R_0603_1608Metric, symbol Device:R_Small
- added R5: 33k2, Resistor_SMD:R_0603_1608Metric, symbol Device:R_Small
- added U3: ~, Package_TO_SOT_SMD:SOT-23-6, symbol Marijn:TPS563201DDCR
Connections:
- new net: D69.1 (K), FB1.1, Q1.2 (S)
- new net: D69.2 (A), Q1.1 (G), R4.1
- new net +3V3: C18.1, C19.1, L2.2, R5.2
- new net +5V: Q1.3 (D)
- new net BUCK_BST: C17.2, U3.6 (VBST)
- new net BUCK_EN: C15.1, C16.1, FB1.2, U3.3 (VIN), U3.5 (EN)
- new net BUCK_FB: R5.1, R6.2, U3.4 (VFB)
- new net BUCK_SW: C17.1, L2.1, U3.2 (SW)
- new net GND: C15.2, C16.2, C18.2, C19.2, R4.2, R6.1, U3.1 (GND)
Other:
- note added: "TODO: fuse?"

Commit message: 65% PCB layout!
Parts:
- FB1: footprint (none) -> Inductor_SMD:L_0805_2012Metric
Other:
- moved on the sheet: C15, C16
Changed lines of the file:
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@@
 	)
 	(junction
-		(at 63.5 34.29)
+		(at 64.77 34.29)
 		(diameter 0)
 		(color 0 0 0 0)
@@
 	)
 	(junction
-		(at 59.69 44.45)
+		(at 60.96 44.45)
 		(diameter 0)
 		(color 0 0 0 0)
@@
 	)
 	(junction
-		(at 59.69 34.29)
+		(at 60.96 34.29)
 		(diameter 0)
 		(color 0 0 0 0)
@@
 	(wire
 		(pts
-			(xy 59.69 44.45) (xy 63.5 44.45)
-		)
-		(stroke
-			(width 0)
-			(type default)
-		)
-	)
-	(wire
-		(pts
 			(xy 50.8 34.29) (xy 50.8 35.56)
 		)
@@
 	(wire
 		(pts
-			(xy 59.69 52.07) (xy 59.69 44.45)
+			(xy 60.96 52.07) (xy 60.96 44.45)
 		)
 		(stroke
@@
 	(wire
 		(pts
+			(xy 64.77 34.29) (xy 68.58 34.29)
+		)
+		(stroke
+			(width 0)
+			(type default)
+		)
+	)
+	(wire
+		(pts
 			(xy 64.77 73.66) (xy 64.77 76.2)
 		)
@@
 	(wire
 		(pts
-			(xy 63.5 34.29) (xy 68.58 34.29)
-		)
-		(stroke
-			(width 0)
-			(type default)
-		)
-	)
-	(wire
-		(pts
-			(xy 59.69 34.29) (xy 63.5 34.29)
+			(xy 60.96 44.45) (xy 64.77 44.45)
+		)
+		(stroke
+			(width 0)
+			(type default)
+		)
+	)
+	(wire
+		(pts
+			(xy 60.96 34.29) (xy 64.77 34.29)
 		)
 		(stroke
@@
 	(wire
 		(pts
-			(xy 59.69 41.91) (xy 59.69 44.45)
+			(xy 60.96 41.91) (xy 60.96 44.45)
 		)
 		(stroke
@@
 	(wire
 		(pts
-			(xy 52.07 52.07) (xy 59.69 52.07)
-		)
-		(stroke
-			(width 0)
-			(type default)
-		)
-	)
-	(wire
-		(pts
-			(xy 63.5 44.45) (xy 63.5 41.91)
+			(xy 52.07 52.07) (xy 60.96 52.07)
+		)
+		(stroke
+			(width 0)
+			(type default)
+		)
+	)
+	(wire
+		(pts
+			(xy 64.77 44.45) (xy 64.77 41.91)
 		)
 		(stroke
@@
 	(wire
 		(pts
-			(xy 58.42 34.29) (xy 59.69 34.29)
+			(xy 58.42 34.29) (xy 60.96 34.29)
 		)
 		(stroke
@@
 	(wire
 		(pts
-			(xy 59.69 34.29) (xy 59.69 36.83)
+			(xy 60.96 34.29) (xy 60.96 36.83)
 		)
 		(stroke
@@
 	(wire
 		(pts
-			(xy 63.5 34.29) (xy 63.5 36.83)
+			(xy 64.77 34.29) (xy 64.77 36.83)
 		)
 		(stroke
@@
 	(symbol
 		(lib_id "Device:C_Small")
-		(at 59.69 39.37 0)
+		(at 60.96 39.37 0)
 		(unit 1)
 		(exclude_from_sim no)
@@
 		(dnp no)
 		(property "Reference" "C15"
-			(at 55.372 37.338 0)
+			(at 56.642 37.338 0)
 			(effects
 				(font
@@
 		)
 		(property "Value" "10u"
-			(at 55.626 41.402 0)
+			(at 56.896 41.402 0)
 			(effects
 				(font
@@
 		)
 		(property "Footprint" "Capacitor_SMD:C_1206_3216Metric"
-			(at 59.69 39.37 0)
+			(at 60.96 39.37 0)
 			(effects
 				(font
@@
 		)
 		(property "Datasheet" "~"
-			(at 59.69 39.37 0)
+			(at 60.96 39.37 0)
 			(effects
 				(font
@@
 		)
 		(property "Description" "Unpolarized capacitor, small symbol"
-			(at 59.69 39.37 0)
+			(at 60.96 39.37 0)
 			(effects
 				(font
@@
 		)
 		(property "LCSC" " C13585"
-			(at 59.69 39.37 0)
+			(at 60.96 39.37 0)
 			(effects
 				(font
@@
 	(symbol
 		(lib_id "Device:C_Small")
-		(at 63.5 39.37 0)
+		(at 64.77 39.37 0)
 		(unit 1)
 		(exclude_from_sim no)
@@
 		(dnp no)
 		(property "Reference" "C16"
-			(at 64.262 37.592 0)
+			(at 65.532 37.592 0)
 			(effects
 				(font
@@
 		)
 		(property "Value" "10u"
-			(at 64.516 41.656 0)
+			(at 65.786 41.656 0)
 			(effects
 				(font
@@
 		)
 		(property "Footprint" "Capacitor_SMD:C_1206_3216Metric"
-			(at 63.5 39.37 0)
+			(at 64.77 39.37 0)
 			(effects
 				(font
@@
 		)
 		(property "Datasheet" "~"
-			(at 63.5 39.37 0)
+			(at 64.77 39.37 0)
 			(effects
 				(font
@@
 		)
 		(property "Description" "Unpolarized capacitor, small symbol"
-			(at 63.5 39.37 0)
+			(at 64.77 39.37 0)
 			(effects
 				(font
@@
 		)
 		(property "LCSC" " C13585"
-			(at 63.5 39.37 0)
+			(at 64.77 39.37 0)
 			(effects
 				(font
@@
 			)
 		)
-		(property "Footprint" ""
+		(property "Footprint" "Inductor_SMD:L_0805_2012Metric"
 			(at 55.88 36.068 90)
 			(effects

Commit message: Layout Progress
Other:
- note added: "TODO: different buck converter (less extended parts!)"
Changed lines of the file:
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@@
+		)
+	)
+	(text "TODO: different buck converter (less extended parts!)"
+		(exclude_from_sim no)
+		(at 140.97 59.436 0)
+		(effects
+			(font
+				(size 1.27 1.27)
+			)
 		)
 	)

Commit message: Layout V1
Other:
- note removed: "TODO: different buck converter (less extended parts!)"
Changed lines of the file:
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@@
-		)
-	)
-	(text "TODO: different buck converter (less extended parts!)"
-		(exclude_from_sim no)
-		(at 140.97 59.436 0)
-		(effects
-			(font
-				(size 1.27 1.27)
-			)
 		)
 	)
