File: Keyboard_PCB/power.kicad_sch (KiCad schematic)
At the start: 13 parts, among them Q1 AO3401A

Commit message: LCD-overhead test
Parts:
- removed C15, C16: 10u, Capacitor_SMD:C_1206_3216Metric, symbol Device:C_Small
- removed C17: 100n, Capacitor_SMD:C_1206_3216Metric, symbol Device:C_Small
- removed C18, C19: 22u, Capacitor_SMD:C_1206_3216Metric, symbol Device:C_Small
- removed D69: 10v, Diode_SMD:D_SOD-523, symbol Device:D_Zener_Small
- removed FB1: 600Ω@100MHz, Inductor_SMD:L_0805_2012Metric, symbol Device:FerriteBead_Small
- removed L2: 2u2, Inductor_SMD:L_Changjiang_FNR3015S, symbol Device:L_Small
- removed Q1: AO3401A, Package_TO_SOT_SMD:SOT-23, symbol Transistor_FET:AO3401A
- removed R4, R6: 10k, Resistor_SMD:R_0603_1608Metric, symbol Device:R_Small
- removed R5: 33k2, Resistor_SMD:R_0603_1608Metric, symbol Device:R_Small
- removed U3: ~, Package_TO_SOT_SMD:SOT-23-6, symbol Marijn:TPS563201DDCR
Other:
- note removed: "TODO: fuse?"
