File: Keyboard_PCB/usb_pwr.kicad_sch (KiCad schematic)
At the start: 45 parts, among them J2 USB-C 16P, U2 ISL91127IR, U3 USBLC6-2SC6, U4 ISL91127IR, U5 MCP73833, U6 MCP73833

Commit message: Cleanup
Other:
- note added: "AMI-MF"
Changed lines of the file:
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@@
+		)
+	)
+	(text "AMI-MF"
+		(exclude_from_sim no)
+		(at 67.818 129.794 0)
+		(effects
+			(font
+				(size 1.27 1.27)
+			)
 		)
 	)
@@
 		(effects
 			(font
+				(size 1.27 1.27)
+			)
+		)
+	)
+	(text "AMI-MF"
+		(exclude_from_sim no)
+		(at 67.818 184.404 0)
+		(effects
+			(font
